File: mcu/eagle_files/mcu_block.sch (EAGLE design)
At the start: 27 parts

Commit message: add buttons
Parts:
- added C4: 0.1uF, SparkFun-Capacitors:CAP0603-CAP
- added R5, R6, R7, R8: 4.7K, SparkFun-Passives:RESISTOR0603-RES
- added U$2, U$3, U$4, U$5: EVQ_TAC_BUTTONS, TuansLib:EVQ_TAC_BUTTONS
- added U$6: 8B_SHIFT_REG, TuansLib:8B_SHIFT_REG
Connections:
- new net N$20: R6.2, U$5.A, U$6.A
- new net N$22: R5.2, U$2.A, U$6.B
- new net N$24: R7.2, U$3.A, U$6.C
- new net N$26: R8.2, U$4.A, U$6.D
- new net SHIFT: U$1.P1.0/TA0CLK/ACLK, U$6.SH/~LD
- net DGND: now also C4.2, R5.1, R6.1, R7.1, R8.1, U$6.GND, U$6.SER
- net SPI_CLK: now also U$6.CLK
- net SPI_MISO: now also U$6.QH
- net SPI_STE: now also U$6.CLK_INH
- net VCC: now also C4.1, U$2.B, U$3.B, U$4.B, U$5.B, U$6.VCC
