File: mainboard/rev0/mainboard.sch (EAGLE design)
At the start: 85 parts, among them Q1 MOSFET-NCHANNEL2N7002PW, Q2 MOSFET-NCHANNEL2N7002PW, Q3 MOSFET-NCHANNEL2N7002PW, Q4 BSS84, Q5 BSS84, Q7 MOSFET-NCHANNEL2N7002PW

Commit message: stuff and things were updated
Connections:
- new net SPYBY_RST: JP1.D+, U$1.RST/NMI/SBWTDIO
- new net SPYBY_TEST: JP1.D-, U$1.TEST/SBWTCK
Changed lines of the file:
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@@
+</segment>
+</net>
+<net name="SPYBY_RST" class="0">
+<segment>
+<pinref part="U$1" gate="G$1" pin="RST/NMI/SBWTDIO"/>
+<wire x1="40.64" y1="40.64" x2="48.26" y2="40.64" width="0.1524" layer="91"/>
+<label x="48.26" y="40.64" size="1.778" layer="95"/>
+</segment>
+<segment>
+<pinref part="JP1" gate="G$1" pin="D+"/>
+<wire x1="-292.1" y1="20.32" x2="-281.94" y2="20.32" width="0.1524" layer="91"/>
+<label x="-281.94" y="20.32" size="1.778" layer="95"/>
+</segment>
+</net>
+<net name="SPYBY_TEST" class="0">
+<segment>
+<pinref part="U$1" gate="G$1" pin="TEST/SBWTCK"/>
+<wire x1="40.64" y1="38.1" x2="48.26" y2="38.1" width="0.1524" layer="91"/>
+<label x="48.26" y="38.1" size="1.778" layer="95"/>
+</segment>
+<segment>
+<pinref part="JP1" gate="G$1" pin="D-"/>
+<wire x1="-292.1" y1="17.78" x2="-281.94" y2="17.78" width="0.1524" layer="91"/>
+<label x="-281.94" y="17.78" size="1.778" layer="95"/>
 </segment>
 </net>

Commit message: deleted some NC parts
Parts:
- removed D4: (no value), SparkFun-DiscreteSemi:DIODEHV
- removed L1: (no value), SparkFun-Passives:INDUCTOR-B82462G
- removed R16, R27: (no value), SparkFun-Passives:RESISTOR0402-RES
- added D9: (no value), SparkFun-DiscreteSemi:DIODESOD523
- added U$11: ASPI-0428S-100M-T, TuansLib:ASPI-0428S-100M-T
Connections:
- removed net N$25: R27.2, U$8.ADC_IN
- removed net N$53: Q4.S, R13.2
- new net N$8: Q4.D, R13.2
- net BORDER: no longer R27.1
- net GND: no longer R16.1
- net N$3: now also D9.C; no longer D4.C
- net N$47: now also U$10.DRAIN; no longer R16.2, U$10.SOURCE
- net N$6: now also U$11.P$1; no longer L1.1
- net VCC: now also U$10.SOURCE, U$11.P$2; no longer L1.2, U$10.DRAIN
- net VCC_T: now also Q4.S; no longer Q4.D
- net VUSB: now also D9.A; no longer D4.A
Other:
- moved on the sheet: Q4

Commit message: updated some values
Parts:
- C1, C27, C28, C29: value (none) -> 0.1uF
- C2: value (none) -> 10uF
- C30: value (none) -> 0.47uF
- L1: value ASPI-0428S-100M-T -> 10uH
- R1: value (none) -> 56K
- R2, R6: value (none) -> 10K
- R3, R4: value (none) -> 1.5K
- R5: value (none) -> 1.6K
- renumbered U$11 to L1
Other:
- note added: "10uH"
- note added: "L1"
- note removed: "add AP2305"
Changed lines of the file:
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@@
 <layer number="102" name="Vscore" color="7" fill="1" visible="no" active="yes"/>
 <layer number="103" name="tMap" color="7" fill="1" visible="no" active="yes"/>
-<layer number="104" name="Name" color="16" fill="1" visible="no" active="yes"/>
+<layer number="104" name="Name" color="16" fill="1" visible="yes" active="yes"/>
 <layer number="105" name="tPlate" color="7" fill="1" visible="no" active="yes"/>
 <layer number="106" name="bPlate" color="7" fill="1" visible="no" active="yes"/>
@@
 <part name="JP1" library="SparkFun-Connectors" deviceset="USB" device="-MICROB"/>
 <part name="SUPPLY4" library="supply2" deviceset="GND" device=""/>
-<part name="C1" library="SparkFun-Capacitors" deviceset="CAP" device="0402-CAP"/>
-<part name="R1" library="SparkFun-Passives" deviceset="RESISTOR" device="0402-RES"/>
-<part name="R2" library="SparkFun-Passives" deviceset="RESISTOR" device="0402-RES"/>
-<part name="R3" library="SparkFun-Passives" deviceset="RESISTOR" device="0402-RES"/>
-<part name="R4" library="SparkFun-Passives" deviceset="RESISTOR" device="0402-RES"/>
-<part name="R5" library="SparkFun-Passives" deviceset="RESISTOR" device="0402-RES"/>
-<part name="C2" library="SparkFun-Capacitors" deviceset="CAP" device="0402-CAP"/>
+<part name="C1" library="SparkFun-Capacitors" deviceset="CAP" device="0402-CAP" value="0.1uF"/>
+<part name="R1" library="SparkFun-Passives" deviceset="RESISTOR" device="0402-RES" value="56K"/>
+<part name="R2" library="SparkFun-Passives" deviceset="RESISTOR" device="0402-RES" value="10K"/>
+<part name="R3" library="SparkFun-Passives" deviceset="RESISTOR" device="0402-RES" value="1.5K"/>
+<part name="R4" library="SparkFun-Passives" deviceset="RESISTOR" device="0402-RES" value="1.5K"/>
+<part name="R5" library="SparkFun-Passives" deviceset="RESISTOR" device="0402-RES" value="1.6K"/>
+<part name="C2" library="SparkFun-Capacitors" deviceset="CAP" device="0402-CAP" value="10uF"/>
 <part name="SUPPLY5" library="supply2" deviceset="GND" device=""/>
 <part name="SUPPLY6" library="supply2" deviceset="GND" device=""/>
-<part name="R6" library="SparkFun-Passives" deviceset="RESISTOR" device="0402-RES"/>
+<part name="R6" library="SparkFun-Passives" deviceset="RESISTOR" device="0402-RES" value="10K"/>
 <part name="D1" library="SparkFun-LED" deviceset="LED-BLUE" device="0603" value="BLUE"/>
 <part name="D2" library="SparkFun-LED" deviceset="LED-BLUE" device="0603" value="BLUE"/>
@@
 <part name="JP3" library="SparkFun-Connectors" deviceset="M03" device="PTH"/>
 <part name="C26" library="SparkFun-Capacitors" deviceset="CAP" device="0402-CAP"/>
-<part name="C27" library="SparkFun-Capacitors" deviceset="CAP" device="0402-CAP"/>
+<part name="C27" library="SparkFun-Capacitors" deviceset="CAP" device="0402-CAP" value="0.1uF"/>
 <part name="SUPPLY25" library="supply2" deviceset="GND" device=""/>
 <part name="SUPPLY26" library="supply2" deviceset="GND" device=""/>
@@
 <part name="R25" library="SparkFun-Passives" deviceset="RESISTOR" device="0402-RES"/>
 <part name="R26" library="SparkFun-Passives" deviceset="RESISTOR" device="0402-RES"/>
-<part name="C28" library="SparkFun-Capacitors" deviceset="CAP" device="0402-CAP"/>
-<part name="C29" library="SparkFun-Capacitors" deviceset="CAP" device="0402-CAP"/>
-<part name="C30" library="SparkFun-Capacitors" deviceset="CAP" device="0402-CAP"/>
+<part name="C28" library="SparkFun-Capacitors" deviceset="CAP" device="0402-CAP" value="0.1uF"/>
+<part name="C29" library="SparkFun-Capacitors" deviceset="CAP" device="0402-CAP" value="0.1uF"/>
+<part name="C30" library="SparkFun-Capacitors" deviceset="CAP" device="0402-CAP" value="0.47uF"/>
 <part name="SUPPLY28" library="supply2" deviceset="GND" device=""/>
 <part name="SUPPLY29" library="supply2" deviceset="GND" device=""/>
-<part name="U$11" library="TuansLib" deviceset="ASPI-0428S-100M-T" device=""/>
+<part name="L1" library="TuansLib" deviceset="ASPI-0428S-100M-T" device="" value="10uH"/>
 <part name="D9" library="SparkFun-DiscreteSemi" deviceset="DIODE" device="SOD523"/>
 </parts>
@@
 <wire x1="-485.14" y1="-68.58" x2="-332.74" y2="-68.58" width="0.1524" layer="97"/>
 <text x="-485.14" y="58.42" size="5.08" layer="97">PWR Monitoring</text>
-<text x="187.96" y="40.64" size="1.778" layer="97">add AP2305</text>
+<text x="-170.18" y="33.02" size="1.778" layer="96">10uH</text>
+<text x="-170.18" y="25.4" size="1.778" layer="96">L1</text>
 </plain>
 <instances>
@@
 <instance part="SUPPLY28" gate="GND" x="-68.58" y="22.86"/>
 <instance part="SUPPLY29" gate="GND" x="-81.28" y="25.4"/>
-<instance part="U$11" gate="G$1" x="-167.64" y="30.48"/>
+<instance part="L1" gate="G$1" x="-167.64" y="30.48"/>
 <instance part="D9" gate="G$1" x="-182.88" y="-10.16" rot="R180"/>
 </instances>
@@
 <wire x1="-190.5" y1="12.7" x2="-187.96" y2="12.7" width="0.1524" layer="91"/>
 <wire x1="-187.96" y1="12.7" x2="-187.96" y2="30.48" width="0.1524" layer="91"/>
-<pinref part="U$11" gate="G$1" pin="P$1"/>
+<pinref part="L1" gate="G$1" pin="P$1"/>
 <wire x1="-187.96" y1="30.48" x2="-177.8" y2="30.48" width="0.1524" layer="91"/>
 </segment>
@@
 <label x="-119.38" y="30.48" size="1.778" layer="95"/>
 <junction x="-127" y="30.48"/>
-<pinref part="U$11" gate="G$1" pin="P$2"/>
+<pinref part="L1" gate="G$1" pin="P$2"/>
 <wire x1="-157.48" y1="30.48" x2="-144.78" y2="30.48" width="0.1524" layer="91"/>
 <junction x="-144.78" y="30.48"/>
