File: mainboard/rev0/mainboard.sch (EAGLE design)
At the start: 83 parts, among them Q1 MOSFET-NCHANNEL2N7002PW, Q2 MOSFET-NCHANNEL2N7002PW, Q3 MOSFET-NCHANNEL2N7002PW, Q4 BSS84, Q5 BSS84, Q7 MOSFET-NCHANNEL2N7002PW

Commit message: ladidadida
Parts:
- C22, C23, C24: value (none) -> 0.1uF
- C25: value (none) -> 0.47uF
- R18: value (none) -> 0.01
- R19, R20, R22: value (none) -> 10K
- R21: value (none) -> 1.8M
Changed lines of the file:
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@@
 <part name="U$9" library="TuansLib" deviceset="BQ27410" device=""/>
 <part name="SUPPLY20" library="supply2" deviceset="GND" device=""/>
-<part name="C22" library="SparkFun-Capacitors" deviceset="CAP" device="0402-CAP"/>
-<part name="C23" library="SparkFun-Capacitors" deviceset="CAP" device="0402-CAP"/>
-<part name="R18" library="SparkFun-Passives" deviceset="RESISTOR" device="0402-RES"/>
-<part name="R19" library="SparkFun-Passives" deviceset="RESISTOR" device="0402-RES"/>
-<part name="R20" library="SparkFun-Passives" deviceset="RESISTOR" device="0402-RES"/>
-<part name="R21" library="SparkFun-Passives" deviceset="RESISTOR" device="0402-RES"/>
+<part name="C22" library="SparkFun-Capacitors" deviceset="CAP" device="0402-CAP" value="0.1uF"/>
+<part name="C23" library="SparkFun-Capacitors" deviceset="CAP" device="0402-CAP" value="0.1uF"/>
+<part name="R18" library="SparkFun-Passives" deviceset="RESISTOR" device="0402-RES" value="0.01"/>
+<part name="R19" library="SparkFun-Passives" deviceset="RESISTOR" device="0402-RES" value="10K"/>
+<part name="R20" library="SparkFun-Passives" deviceset="RESISTOR" device="0402-RES" value="10K"/>
+<part name="R21" library="SparkFun-Passives" deviceset="RESISTOR" device="0402-RES" value="1.8M"/>
 <part name="SUPPLY21" library="supply2" deviceset="GND" device=""/>
 <part name="SUPPLY22" library="supply2" deviceset="GND" device=""/>
-<part name="R22" library="SparkFun-Passives" deviceset="RESISTOR" device="0402-RES"/>
-<part name="C24" library="SparkFun-Capacitors" deviceset="CAP" device="0402-CAP"/>
-<part name="C25" library="SparkFun-Capacitors" deviceset="CAP" device="0402-CAP"/>
+<part name="R22" library="SparkFun-Passives" deviceset="RESISTOR" device="0402-RES" value="10K"/>
+<part name="C24" library="SparkFun-Capacitors" deviceset="CAP" device="0402-CAP" value="0.1uF"/>
+<part name="C25" library="SparkFun-Capacitors" deviceset="CAP" device="0402-CAP" value="0.47uF"/>
 <part name="U$10" library="TuansLib" deviceset="DMG2305UX" device=""/>
 <part name="SUPPLY23" library="supply2" deviceset="GND" device=""/>
