File: mainboard/rev0/mainboard.brd (EAGLE design)
At the start: 43.2 x 38.1 mm, 58 parts, among them Q1 MOSFET-NCHANNEL2N7002PW, Q2 MOSFET-NCHANNEL2N7002PW, Q3 MOSFET-NCHANNEL2N7002PW, Q4 MOSFET-NCHANNEL2N7002PW, Q5 BSS84, Q6 BSS84, Q7 MOSFET-NCHANNEL2N7002PW

Commit message: rarrrrrarararaaawww.
Parts:
- removed Q6: BSS84, transistor-small-signal:SOT23
- added C21, C22, C23, C24, C25, C26, C27, C28, C29, C30: (no value), SparkFun-Capacitors:0402-CAP
- added D5, D6, D7, D8: BLUE, SparkFun-LED:LED-0603
- added JP2: M02PTH, SparkFun-Connectors:1X02
- added JP3: (no value), SparkFun-Connectors:1X03
- added R18, R19, R20, R21, R22, R23, R24, R25, R26, R27: (no value), SparkFun-Passives:0402-RES
- added U$10: DMG2305UX, TuansLib:SOT23
- added U$9: BQ27410, TuansLib:SON_DRZ_12PIN
- Q4: value MOSFET-NCHANNEL2N7002PW -> BSS84; device SparkFun-DiscreteSemi:SOT323 -> transistor-small-signal:SOT23
- moved Q4 63.6 mm to (-50.8, -213.4)
- moved L1 5.68 mm to (30.5, 12.7), flipped to the bottom
- moved JP1 5.08 mm to (38.1, 11.4)
- moved U$1 2.54 mm to (22.9, 8.89)
- moved U$3 2.54 mm to (34.3, 6.35), flipped to the top, turned to 180 degrees
- moved U$7 1.44 mm to (37.8, 34.0)
- moved U$6 1.27 mm to (37.8, 1.78)
Connections:
- removed net N$17: R7.1
- removed net N$18: R8.1
- removed net N$19: R9.1
- removed net N$20: R10.1
- removed net N$21: U$8.4
- removed net N$22: U$8.5
- removed net N$23: U$8.6
- removed net N$24: U$8.7
- removed net N$8: U$8.2
- removed net SPI_STE: U$1.41
- new net BTN_0: R7.1, U$1.26
- new net BTN_1: R8.1, U$1.27
- new net BTN_2: R9.1, U$1.28
- new net BTN_3: R10.1, U$1.29
- new net EPD_BUSY: U$1.5, U$8.2
- new net EPD_CS: U$1.3, U$8.1
- new net EPD_RST: U$1.6, U$8.7
- new net LED_0: D5.C, U$1.30
- new net LED_1: D6.C, U$1.31
- new net LED_2: D7.C, U$1.32
- new net LED_3: D8.C, U$1.33
- new net N$48: D5.A, R23.1
- new net N$51: D6.A, R24.1
- new net N$54: C23.1, R18.1, U$9.7
- new net N$55: D7.A, R25.1
- new net N$56: D8.A, R26.1
- new net PM_BIN: R21.2, U$1.37, U$9.1
- new net PM_GPOUT: R22.2, U$1.36, U$9.12
- new net PM_SCL: R19.2, U$1.35, U$9.11
- new net PM_SDA: R20.2, U$1.34, U$9.10
- new net SENSOR_DATA: JP3.2, U$1.1, U$1.2
- new net VCC_R: C25.1, U$9.2, U$9.5
- net BATT_PWR: now also C22.1, C24.1, JP2.2, U$9.3, U$9.4
- net BORDER: now also R27.1
- net EPD_BORDER: now also U$1.7
- net EPD_DISCHARGE: now also U$1.8
- net EPD_PANEL: now also U$1.4
- net EPD_PWM: now also U$1.19
- net GND: now also C21.2, C22.2, C23.2, C24.2, C25.2, C26.2, C27.2, C28.2, C29.2, C30.1, JP2.1, JP3.1, R18.2, U$9.13, U$9.6, U$9.8, U$9.9, U$9.P$15, U$9.P$16, U$9.P$17, U$9.P$18, U$9.P$19, U$9.P$20
- net N$25: now also R27.2
- net N$47: now also U$10.2; no longer Q6.3
- net N$50: now also U$10.1; no longer Q6.1
- net N$53: now also Q4.2; no longer Q4.3
- net N$7: now also C30.2, U$1.17; no longer U$8.1
- net SPI_CLK: now also U$8.4
- net SPI_MISO: now also U$8.6
- net SPI_MOSI: now also U$8.5
- net VCC: now also C26.1, C27.1, C28.1, C29.1, JP3.3, R19.1, R20.1, R21.1, R22.1, R23.2, R24.2, R25.2, R26.2, U$1.11, U$1.15, U$1.40, U$10.3; no longer Q6.2
- net VCC_T: now also Q4.3; no longer Q4.2
- net VCOM: now also C21.1
- net VCOM_DRIVER: now also R11.1

Commit message: stuff and things were updated
Parts:
- moved C29 318.9 mm to (14.2, 21.3)
- moved R27 316.3 mm to (3.56, 26.7)
- moved C27 315.8 mm to (35.6, 35.6), flipped to the bottom, turned to 270 degrees
- moved C28 304.5 mm to (15.5, 8.38)
- moved R26 296.9 mm to (27.7, 1.27), turned to 180 degrees
- moved JP2 292.4 mm to (38.1, 25.4), turned to 90 degrees
- moved R25 292.2 mm to (20.8, 1.27), turned to 180 degrees
- moved R24 287.6 mm to (14.2, 1.27), turned to 180 degrees
- moved D8 287.0 mm to (30.5, 1.27), turned to 270 degrees
- moved R23 283.1 mm to (7.37, 1.27), turned to 180 degrees
- moved D7 282.7 mm to (23.7, 1.27), turned to 270 degrees
- moved C26 281.9 mm to (31.8, 3.81), turned to 270 degrees
- moved D6 278.9 mm to (16.9, 1.27), turned to 270 degrees
- moved C24 278.4 mm to (35.8, 26.7), turned to 270 degrees
- moved JP3 275.9 mm to (34.0, 1.78), turned to 90 degrees
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Connections:
- new net SPYBY_RST: JP1.D+, U$1.64
- new net SPYBY_TEST: JP1.D-, U$1.59

Commit message: Finished the routing and shipped the board out
Parts:
- removed D4: (no value), SparkFun-DiscreteSemi:DIODE-HV
- removed L1: (no value), SparkFun-Passives:B82462G
- removed R16, R27: (no value), SparkFun-Passives:0402-RES
- added D9: (no value), SparkFun-DiscreteSemi:SOD523
- added U$11: ASPI-0428S-100M-T, TuansLib:ASPI_0428S-100M-T
- moved C30 312.4 mm to (30.5, 6.60), turned to 90 degrees
- moved C25 277.0 mm to (39.4, 21.3), turned to 270 degrees
- moved U$10 265.5 mm to (15.2, 11.9)
- moved R18 259.0 mm to (32.0, 20.1), turned to 90 degrees
- moved C23 257.0 mm to (33.3, 20.1), turned to 90 degrees
- moved Q4 225.9 mm to (10.7, 4.06), turned to 90 degrees
- moved C20 223.2 mm to (13.7, 16.3), turned to 90 degrees
- moved R17 219.3 mm to (12.2, 17.8), turned to 270 degrees
- moved C19 217.8 mm to (9.40, 14.5), turned to 180 degrees
- moved Q7 214.3 mm to (10.9, 8.89), turned to 180 degrees
- moved C21 213.1 mm to (5.56, 4.11), turned to 270 degrees
- moved R15 211.7 mm to (9.40, 15.7), turned to 180 degrees
- moved C14 197.2 mm to (14.5, 16.8), flipped to the bottom
- moved Q5 192.0 mm to (15.2, 6.86)
- moved D3 186.3 mm to (10.7, 12.4), flipped to the bottom, turned to 90 degrees
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Connections:
- removed net N$25: R27.2, U$8.8
- removed net N$53: Q4.2, R13.2
- new net N$8: Q4.3, R13.2
- net BORDER: no longer R27.1
- net GND: no longer R16.1
- net N$3: now also D9.C; no longer D4.C
- net N$47: now also U$10.3; no longer R16.2, U$10.2
- net N$6: now also U$11.1; no longer L1.P$1
- net VCC: now also U$10.2, U$11.2; no longer L1.P$2, U$10.3
- net VCC_T: now also Q4.2; no longer Q4.3
- net VUSB: now also D9.A; no longer D4.A
Routing:
- net GND: track 0.00 -> 272.9 mm, vias 0 -> 12
- net VCC: track 0.00 -> 129.8 mm, vias 0 -> 8
- net N$3: track 0.00 -> 48.9 mm, vias 0 -> 5
- net PM_BIN: track 0.00 -> 47.1 mm, vias 0 -> 2
- net BTN_0: track 0.00 -> 47.0 mm, vias 0 -> 3
- net BTN_1: track 0.00 -> 44.0 mm, vias 0 -> 3
- net EPD_BUSY: track 0.00 -> 38.5 mm, vias 0 -> 5
- net N$11: track 0.00 -> 37.5 mm, vias 0 -> 1
- net LED_0: track 0.00 -> 37.1 mm
- net SPYBY_TEST: track 0.00 -> 36.0 mm, vias 0 -> 3
- net VUSB: track 0.00 -> 34.4 mm, vias 0 -> 5
- net EPD_RST: track 0.00 -> 34.3 mm, vias 0 -> 5
- net EPD_CS: track 0.00 -> 33.2 mm, vias 0 -> 3
- net LED_1: track 0.00 -> 30.8 mm, vias 0 -> 2
- net SPI_MOSI: track 0.00 -> 29.0 mm, vias 0 -> 5
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Other:
- board size 43.2 x 38.1 mm -> 40.6 x 38.1 mm

Commit message: ladidadida
Parts:
- C1, C22, C23, C24, C27, C28, C29: value (none) -> 0.1uF
- C2: value (none) -> 10uF
- C25, C30: value (none) -> 0.47uF
- L1: value ASPI-0428S-100M-T -> 10uH
- R1: value (none) -> 56K
- R18: value (none) -> 0.01
- R19, R2, R20, R22, R6: value (none) -> 10K
- R21: value (none) -> 1.8M
- R3, R4: value (none) -> 1.5K
- R5: value (none) -> 1.6K
- renumbered U$11 to L1
Changed lines of the file:
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@@
 <wire x1="40.64" y1="38.1" x2="0" y2="38.1" width="0" layer="20"/>
 <wire x1="0" y1="38.1" x2="0" y2="0" width="0" layer="20"/>
-<dimension x1="40.64" y1="0" x2="40.64" y2="38.1" x3="48.26" y3="19.05" textsize="1.778" layer="20" unit="mil"/>
-<dimension x1="40.64" y1="38.1" x2="0" y2="38.1" x3="20.32" y3="45.72" textsize="1.778" layer="20" unit="mil"/>
+<dimension x1="40.64" y1="0" x2="40.64" y2="38.1" x3="48.26" y3="19.05" textsize="1.778" layer="47" unit="mil"/>
+<dimension x1="40.64" y1="38.1" x2="0" y2="38.1" x3="20.32" y3="45.72" textsize="1.778" layer="47" unit="mil"/>
 </plain>
 <attributes>
@@
 <attribute name="PROD_ID" value="CONN-09505" x="39.116" y="11.176" size="1.778" layer="28" rot="MR270" display="off"/>
 </element>
-<element name="C1" library="SparkFun-Capacitors" package="0402-CAP" value="" x="33.6804" y="11.3792" rot="MR270"/>
-<element name="R1" library="SparkFun-Passives" package="0402-RES" value="" x="22.86" y="29.718" rot="R90"/>
-<element name="R2" library="SparkFun-Passives" package="0402-RES" value="" x="23.876" y="27.432" rot="R180"/>
-<element name="R3" library="SparkFun-Passives" package="0402-RES" value="" x="38.862" y="18.542" rot="MR90"/>
-<element name="R4" library="SparkFun-Passives" package="0402-RES" value="" x="38.862" y="21.844" rot="MR90"/>
-<element name="R5" library="SparkFun-Passives" package="0402-RES" value="" x="30.226" y="34.6964" rot="R180"/>
-<element name="C2" library="SparkFun-Capacitors" package="0402-CAP" value="" x="21.336" y="29.718" rot="R270"/>
-<element name="R6" library="SparkFun-Passives" package="0402-RES" value="" x="25.908" y="33.274"/>
+<element name="C1" library="SparkFun-Capacitors" package="0402-CAP" value="0.1uF" x="33.6804" y="11.3792" rot="MR270"/>
+<element name="R1" library="SparkFun-Passives" package="0402-RES" value="56K" x="22.86" y="29.718" rot="R90"/>
+<element name="R2" library="SparkFun-Passives" package="0402-RES" value="10K" x="23.876" y="27.432" rot="R180"/>
+<element name="R3" library="SparkFun-Passives" package="0402-RES" value="1.5K" x="38.862" y="18.542" rot="MR90"/>
+<element name="R4" library="SparkFun-Passives" package="0402-RES" value="1.5K" x="38.862" y="21.844" rot="MR90"/>
+<element name="R5" library="SparkFun-Passives" package="0402-RES" value="1.6K" x="30.226" y="34.6964" rot="R180"/>
+<element name="C2" library="SparkFun-Capacitors" package="0402-CAP" value="10uF" x="21.336" y="29.718" rot="R270"/>
+<element name="R6" library="SparkFun-Passives" package="0402-RES" value="10K" x="25.908" y="33.274"/>
 <element name="D1" library="SparkFun-LED" package="LED-0603" value="BLUE" x="40.132" y="21.844" rot="MR0">
 <attribute name="PROD_ID" value="DIO-08575" x="40.132" y="21.844" size="1.778" layer="28" rot="MR0" display="off"/>
@@
 <element name="Q4" library="transistor-small-signal" package="SOT23" value="BSS84" x="10.668" y="4.064" rot="R90"/>
 <element name="U$9" library="TuansLib" package="SON_DRZ_12PIN" value="BQ27410" x="37.846" y="22.098" rot="R180"/>
-<element name="C22" library="SparkFun-Capacitors" package="0402-CAP" value="" x="34.544" y="26.67" rot="R270"/>
-<element name="C23" library="SparkFun-Capacitors" package="0402-CAP" value="" x="33.274" y="20.066" rot="R90"/>
-<element name="R18" library="SparkFun-Passives" package="0402-RES" value="" x="32.004" y="20.066" rot="R90"/>
-<element name="R19" library="SparkFun-Passives" package="0402-RES" value="" x="29.464" y="20.828" rot="R270"/>
-<element name="R20" library="SparkFun-Passives" package="0402-RES" value="" x="30.734" y="20.828" rot="R270"/>
-<element name="R21" library="SparkFun-Passives" package="0402-RES" value="" x="26.924" y="20.828" rot="R270"/>
-<element name="R22" library="SparkFun-Passives" package="0402-RES" value="" x="28.194" y="20.828" rot="R270"/>
-<element name="C24" library="SparkFun-Capacitors" package="0402-CAP" value="" x="35.814" y="26.67" rot="R270"/>
-<element name="C25" library="SparkFun-Capacitors" package="0402-CAP" value="" x="39.37" y="21.336" rot="R270"/>
+<element name="C22" library="SparkFun-Capacitors" package="0402-CAP" value="0.1uF" x="34.544" y="26.67" rot="R270"/>
+<element name="C23" library="SparkFun-Capacitors" package="0402-CAP" value="0.1uF" x="33.274" y="20.066" rot="R90"/>
+<element name="R18" library="SparkFun-Passives" package="0402-RES" value="0.01" x="32.004" y="20.066" rot="R90"/>
+<element name="R19" library="SparkFun-Passives" package="0402-RES" value="10K" x="29.464" y="20.828" rot="R270"/>
+<element name="R20" library="SparkFun-Passives" package="0402-RES" value="10K" x="30.734" y="20.828" rot="R270"/>
+<element name="R21" library="SparkFun-Passives" package="0402-RES" value="1.8M" x="26.924" y="20.828" rot="R270"/>
+<element name="R22" library="SparkFun-Passives" package="0402-RES" value="10K" x="28.194" y="20.828" rot="R270"/>
+<element name="C24" library="SparkFun-Capacitors" package="0402-CAP" value="0.1uF" x="35.814" y="26.67" rot="R270"/>
+<element name="C25" library="SparkFun-Capacitors" package="0402-CAP" value="0.47uF" x="39.37" y="21.336" rot="R270"/>
 <element name="U$10" library="TuansLib" package="SOT23" value="DMG2305UX" x="15.24" y="11.938"/>
 <element name="JP2" library="SparkFun-Connectors" package="1X02" value="M02PTH" x="39.37" y="25.4" rot="R90"/>
 <element name="JP3" library="SparkFun-Connectors" package="1X03" value="" x="34.036" y="1.778" rot="R90"/>
 <element name="C26" library="SparkFun-Capacitors" package="0402-CAP" value="" x="31.75" y="3.81" rot="MR270"/>
-<element name="C27" library="SparkFun-Capacitors" package="0402-CAP" value="" x="39.116" y="35.56" rot="MR270"/>
+<element name="C27" library="SparkFun-Capacitors" package="0402-CAP" value="0.1uF" x="39.116" y="35.56" rot="MR270"/>
 <element name="D5" library="SparkFun-LED" package="LED-0603" value="BLUE" x="10.16" y="1.016" rot="R270">
 <attribute name="PROD_ID" value="DIO-08575" x="10.16" y="1.016" size="1.778" layer="27" rot="R270" display="off"/>
@@
 <element name="R25" library="SparkFun-Passives" package="0402-RES" value="" x="20.828" y="1.016" rot="R180"/>
 <element name="R26" library="SparkFun-Passives" package="0402-RES" value="" x="27.432" y="1.016" rot="R180"/>
-<element name="C28" library="SparkFun-Capacitors" package="0402-CAP" value="" x="26.162" y="4.826"/>
-<element name="C29" library="SparkFun-Capacitors" package="0402-CAP" value="" x="25.7302" y="18.7198"/>
-<element name="C30" library="SparkFun-Capacitors" package="0402-CAP" value="" x="30.48" y="6.604" rot="R90"/>
-<element name="U$11" library="TuansLib" package="ASPI_0428S-100M-T" value="ASPI-0428S-100M-T" x="32.004" y="21.336" rot="MR180"/>
+<element name="C28" library="SparkFun-Capacitors" package="0402-CAP" value="0.1uF" x="26.162" y="4.826"/>
+<element name="C29" library="SparkFun-Capacitors" package="0402-CAP" value="0.1uF" x="25.7302" y="18.7198"/>
+<element name="C30" library="SparkFun-Capacitors" package="0402-CAP" value="0.47uF" x="30.48" y="6.604" rot="R90"/>
+<element name="L1" library="TuansLib" package="ASPI_0428S-100M-T" value="10uH" x="32.004" y="21.336" rot="MR180"/>
 <element name="D9" library="SparkFun-DiscreteSemi" package="SOD523" value="" x="37.338" y="16.256" rot="MR270"/>
 </elements>
@@
 <signal name="N$6">
 <contactref element="U$3" pad="19"/>
-<contactref element="U$11" pad="1"/>
+<contactref element="L1" pad="1"/>
 <wire x1="26.416" y1="30.9118" x2="27.3558" y2="30.9118" width="0.1524" layer="1"/>
 <wire x1="25.8572" y1="30.353" x2="26.416" y2="30.9118" width="0.1524" layer="1"/>
@@
 <contactref element="C28" pad="1"/>
 <contactref element="U$10" pad="2"/>
-<contactref element="U$11" pad="2"/>
+<contactref element="L1" pad="2"/>
 <wire x1="25.5016" y1="6.35" x2="25.5016" y2="5.969" width="0.1524" layer="1"/>
 <wire x1="25.5016" y1="5.969" x2="25.5016" y2="4.826" width="0.1524" layer="1"/>
