File: mainboard/test/mainboard.sch (EAGLE design)
At the start: 83 parts, among them Q1 MOSFET-NCHANNEL2N7002PW, Q2 MOSFET-NCHANNEL2N7002PW, Q3 MOSFET-NCHANNEL2N7002PW, Q4 BSS84, Q5 BSS84, Q7 MOSFET-NCHANNEL2N7002PW

Commit message: created a back up test board for check off
Parts:
- added TP1, TP10, TP11, TP12, TP13, TP14, TP15, TP16, TP17, TP18, TP19, TP2, TP22, TP23, TP24, TP26, TP27, TP28, TP29, TP3, TP30, TP4, TP5, TP6, TP7, TP8, TP9: TPB1,27, testpad:TPB1,27
Connections:
- net EPD_BORDER: now also TP16.TP
- net EPD_BUSY: now also TP14.TP
- net EPD_CS: now also TP12.TP
- net EPD_DISCHARGE: now also TP17.TP
- net EPD_PANEL: now also TP13.TP
- net EPD_PWM: now also TP10.TP
- net EPD_RST: now also TP15.TP
- net N$5: now also TP2.TP
- net N$6: now also TP1.TP
- net PM_BIN: now also TP6.TP
- net PM_GPOUT: now also TP3.TP
- net PM_SCL: now also TP4.TP
- net PM_SDA: now also TP5.TP
- net SENSOR_DATA: now also TP11.TP
- net SPI_CLK: now also TP22.TP
- net SPI_MISO: now also TP24.TP
- net SPI_MOSI: now also TP23.TP
- net SPYBY_RST: now also TP18.TP
- net SPYBY_TEST: now also TP19.TP
- net UART_RX: now also TP8.TP
- net UART_TX: now also TP9.TP
- net VCC_R: now also TP7.TP
- net VCC_T: now also TP30.TP
- net VDH: now also TP28.TP
- net VDL: now also TP29.TP
- net VGH: now also TP26.TP
- net VGL: now also TP27.TP
