File: mainboard/rev1/mainboard.brd (EAGLE design)
At the start: 40.6 x 30.5 mm, 82 parts, among them Q1 MOSFET-NCHANNEL2N7002PW, Q2 MOSFET-NCHANNEL2N7002PW, Q3 MOSFET-NCHANNEL2N7002PW, Q4 BSS84, Q5 BSS84, Q6 MOSFET-NCHANNEL2N7002PW, Q7 MOSFET-NCHANNEL2N7002PW, X1 CRYSTAL"32.768"

Commit message: routed
Parts:
- removed U$13: SWITCH_SLIDEMICRO_SWITCH, TuansLib:JS2202011AQN
- moved U$12 24.4 mm to (16.4, 1.57), turned to 90 degrees
- moved C26 23.8 mm to (13.5, 4.55), flipped to the top, turned to 0 degrees
- moved Q6 20.5 mm to (17.3, 3.53), turned to 180 degrees
- moved X1 13.4 mm to (24.4, 12.8), turned to 270 degrees
- moved Q5 11.3 mm to (7.44, 18.8), turned to 90 degrees
- moved C25 9.02 mm to (29.6, 25.7), turned to 90 degrees
- moved C30 8.36 mm to (28.6, 16.8)
- moved D5 8.13 mm to (28.6, 0.58)
- moved U$10 7.63 mm to (6.60, 5.82)
- moved C31 7.31 mm to (23.2, 8.84), flipped to the top, turned to 270 degrees
- moved R17 7.17 mm to (7.42, 23.6)
- moved L1 7.08 mm to (30.4, 2.97), turned to 90 degrees
- moved C11 6.84 mm to (7.65, 16.8), flipped to the bottom, turned to 270 degrees
- moved R6 6.63 mm to (30.8, 4.55), turned to 180 degrees
- moved Q7 6.34 mm to (9.58, 19.5), flipped to the bottom
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Connections:
- removed net N$20: R6.2, U$13.3, U$13.6
- net BATT_PWR: now also R6.2; no longer U$13.2, U$13.5
Routing:
- net LED_0: track 0.00 -> 92.3 mm, vias 0 -> 2
- net EPD_DISCHARGE: track 76.6 -> 13.1 mm, vias 7 -> 2
- net VCC: track 92.7 -> 153.4 mm, vias 9 -> 6
- net VCC_T: track 65.2 -> 18.7 mm, vias 5 -> 3
- net SENSOR_EN: track 0.00 -> 45.1 mm, vias 0 -> 6
- net BTN_0: track 0.00 -> 33.3 mm, vias 0 -> 6
- net EPD_PWM: track 49.9 -> 17.6 mm, vias 6 -> 5
- net LED_1: track 0.00 -> 31.9 mm, vias 0 -> 4
- net GND: track 269.1 -> 237.9 mm, vias 18 -> 14
- net BTN_1: track 0.00 -> 29.6 mm, vias 0 -> 3
- net BT_BAUD: track 13.4 -> 41.2 mm, vias 1 -> 3
- net BTN_2: track 45.0 -> 22.9 mm, vias 4 -> 2
- net EPD_RST: track 0.00 -> 21.5 mm, vias 0 -> 3
- net VGH: track 28.9 -> 10.4 mm, vias 3 -> 2
- net N$17: track 18.0 -> 0.00 mm
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- added copper zone on layer 16, net GND
Other:
- board size 40.6 x 30.5 mm -> 40.6 x 34.3 mm
