File: mainboard/rev1/mainboard.sch (EAGLE design)
At the start: 82 parts, among them Q1 MOSFET-NCHANNEL2N7002PW, Q2 MOSFET-NCHANNEL2N7002PW, Q3 MOSFET-NCHANNEL2N7002PW, Q4 BSS84, Q5 BSS84, Q6 MOSFET-NCHANNEL2N7002PW, Q7 MOSFET-NCHANNEL2N7002PW, X1 CRYSTAL"32.768"

Commit message: routed
Parts:
- removed U$13: SWITCH_SLIDEMICRO_SWITCH, TuansLib:SWITCH_SLIDEMICRO_SWITCH
Connections:
- removed net N$20: R6.2, U$13.@3
- net BATT_PWR: now also R6.2; no longer U$13.@2
Changed lines of the file:
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@@
 <part name="SUPPLY16" library="supply2" deviceset="GND" device=""/>
 <part name="Q6" library="SparkFun-DiscreteSemi" deviceset="MOSFET-NCHANNEL" device="2N7002PW"/>
-<part name="U$13" library="TuansLib" deviceset="SWITCH_SLIDE" device="MICRO_SWITCH">
-<attribute name="PART#" value="JS202011AQN"/>
-</part>
 <part name="X1" library="TuansLib" deviceset="CRYSTAL" device="&quot;32.768&quot;"/>
 <part name="C31" library="SparkFun-Capacitors" deviceset="CAP" device="0402-CAP" value="12.5pF"/>
@@
 <attribute name="VALUE" x="-403.86" y="-160.02" size="1.778" layer="96" rot="MR0"/>
 </instance>
-<instance part="U$13" gate="G$1" x="-256.54" y="-48.26">
-<attribute name="PART#" x="-256.54" y="-48.26" size="3.81" layer="96" display="off"/>
-</instance>
 <instance part="X1" gate="G$1" x="63.5" y="-7.62"/>
 <instance part="C31" gate="G$1" x="60.96" y="-12.7" smashed="yes" rot="R90">
@@
 </segment>
 <segment>
-<pinref part="U$13" gate="G$1" pin="@2"/>
-<wire x1="-256.54" y1="-53.34" x2="-256.54" y2="-55.88" width="0.1524" layer="91"/>
-<wire x1="-256.54" y1="-55.88" x2="-269.24" y2="-55.88" width="0.1524" layer="91"/>
-<label x="-284.48" y="-55.88" size="1.778" layer="95"/>
+<pinref part="R6" gate="G$1" pin="2"/>
+<wire x1="-241.3" y1="-20.32" x2="-241.3" y2="-35.56" width="0.1524" layer="91"/>
+<label x="-241.3" y="-38.1" size="1.778" layer="95"/>
 </segment>
 </net>
@@
 </segment>
 </net>
-<net name="N$20" class="0">
-<segment>
-<pinref part="U$13" gate="G$1" pin="@3"/>
-<wire x1="-254" y1="-53.34" x2="-254" y2="-55.88" width="0.1524" layer="91"/>
-<pinref part="R6" gate="G$1" pin="2"/>
-<wire x1="-254" y1="-55.88" x2="-241.3" y2="-55.88" width="0.1524" layer="91"/>
-<wire x1="-241.3" y1="-55.88" x2="-241.3" y2="-20.32" width="0.1524" layer="91"/>
-</segment>
-</net>
